File: stepper_driver.sch (KiCad schematic (older format))
At the start: 33 parts, among them P1 PWR_JACK_2.5x5.5_SMD_VERT, P2 BNC, U1 AT42QT2120-MMHR

Commit message: Clear schematic and board
Parts:
- removed C1: 10uF, stepper_driver:SM0805, symbol stepper_driver:10uF
- removed C2: 1uF, stepper_driver:SM0402_POL, symbol stepper_driver:1uF
- removed C3: 0.1uF, stepper_driver:SM0402, symbol stepper_driver:0.1uF
- removed D1: DIODE_SCHOTTKY_45V_10A, stepper_driver:CFP15, symbol stepper_driver:DIODE_SCHOTTKY_45V_10A
- removed D2: DIODE_LOW_REV_CURRENT_0402, stepper_driver:SM0402_POL, symbol stepper_driver:DIODE_LOW_REV_CURRENT_0402
- removed L1: LED_GRN, stepper_driver:LED0805, symbol stepper_driver:LED_GRN
- removed MH1, MH10, MH11, MH12, MH13, MH14, MH2, MH3, MH4, MH5, MH6, MH7, MH8, MH9: MOUNTING_HOLE_4-40, stepper_driver:MOUNTING_HOLE_4-40, symbol stepper_driver:MOUNTING_HOLE_4-40
- removed P1: PWR_JACK_2.5x5.5_SMD_VERT, stepper_driver:DCJACK_3PIN_SMD_VERT, symbol stepper_driver:PWR_JACK_2.5x5.5_SMD_VERT
- removed P2: BNC, stepper_driver:BNC, symbol stepper_driver:BNC
- removed R1, R2, R3: 2.2k, stepper_driver:SM0402, symbol stepper_driver:2.2k
- removed R4, R5: 47k, stepper_driver:SM0402, symbol stepper_driver:47k
- removed TEENSY1: TEENSY_4.0_HEADERS, stepper_driver:TEENSY_4.0_HEADERS, symbol stepper_driver:TEENSY_4.0_HEADERS
- removed U1: AT42QT2120-MMHR, stepper_driver:QFN-20-1EP_3x3mm_P0.45mm_EP1.6x1.6mm, symbol stepper_driver:AT42QT2120-MMHR
Connections:
- net labels removed: GND, LICK_DETECTED, RESET, SCL, SDA, SOLENOID_0, SOLENOID_1, SOLENOID_10, SOLENOID_11, SOLENOID_2, SOLENOID_3, SOLENOID_4, SOLENOID_5, SOLENOID_6, SOLENOID_7, SOLENOID_8, SOLENOID_9, SYNC, TOUCH_0, TOUCH_1, TOUCH_10, TOUCH_11, TOUCH_2, TOUCH_3, TOUCH_4, TOUCH_5, TOUCH_6, TOUCH_7, TOUCH_8, TOUCH_9, VAA, VCC, VDD, Vled, ~CHANGE
- wire segments 165 -> 0
- no-connect marks 24 -> 0

Commit message: Add mounting holes, stepstick, and term block
Parts:
- added MH1, MH2, MH3, MH4: MOUNTING_HOLE_4-40, stepper_driver:MOUNTING_HOLE_4-40, symbol stepper_driver:MOUNTING_HOLE_4-40
- added SS1: STEPSTICK_TMC2209, stepper_driver:STEPSTICK_TMC2209, symbol stepper_driver:STEPSTICK_TMC2209
- added T1: TERM_BLK_4_PIN_0.1_PITCH, stepper_driver:TERM_BLK_4_PIN_0.1_PITCH, symbol stepper_driver:TERM_BLK_4_PIN_0.1_PITCH
Connections:
- no-connect marks 0 -> 24
Changed lines of the file:
@@
 	1    0    0    -1
 $EndComp
+$Comp
+L stepper_driver:MOUNTING_HOLE_4-40 MH1
+U 1 1 6171DD70
+P 9600 750
+F 0 "MH1" H 9659 869 50  0000 L CNN
+F 1 "MOUNTING_HOLE_4-40" H 9659 777 50  0000 L CNN
+F 2 "stepper_driver:MOUNTING_HOLE_4-40" H 9800 750 50  0001 C CNN
+F 3 "" H 9800 750 50  0001 C CNN
+	1    9600 750
+	1    0    0    -1
+$EndComp
+$Comp
+L stepper_driver:MOUNTING_HOLE_4-40 MH2
+U 1 1 6171E6FB
+P 9600 950
+F 0 "MH2" H 9659 1069 50  0000 L CNN
+F 1 "MOUNTING_HOLE_4-40" H 9659 977 50  0000 L CNN
+F 2 "stepper_driver:MOUNTING_HOLE_4-40" H 9800 950 50  0001 C CNN
+F 3 "" H 9800 950 50  0001 C CNN
+	1    9600 950
+	1    0    0    -1
+$EndComp
+$Comp
+L stepper_driver:MOUNTING_HOLE_4-40 MH3
+U 1 1 6171E9F1
+P 9600 1150
+F 0 "MH3" H 9659 1269 50  0000 L CNN
+F 1 "MOUNTING_HOLE_4-40" H 9659 1177 50  0000 L CNN
+F 2 "stepper_driver:MOUNTING_HOLE_4-40" H 9800 1150 50  0001 C CNN
+F 3 "" H 9800 1150 50  0001 C CNN
+	1    9600 1150
+	1    0    0    -1
+$EndComp
+$Comp
+L stepper_driver:MOUNTING_HOLE_4-40 MH4
+U 1 1 6171EA61
+P 9600 1350
+F 0 "MH4" H 9659 1469 50  0000 L CNN
+F 1 "MOUNTING_HOLE_4-40" H 9659 1377 50  0000 L CNN
+F 2 "stepper_driver:MOUNTING_HOLE_4-40" H 9800 1350 50  0001 C CNN
+F 3 "" H 9800 1350 50  0001 C CNN
+	1    9600 1350
+	1    0    0    -1
+$EndComp
+NoConn ~ 9600 750
+NoConn ~ 9600 950
+NoConn ~ 9600 1150
+NoConn ~ 9600 1350
+$Comp
+L stepper_driver:STEPSTICK_TMC2209 SS1
+U 1 1 6172192F
+P 5600 3850
+F 0 "SS1" H 5900 4400 60  0000 C CNN
+F 1 "STEPSTICK_TMC2209" H 6150 3300 60  0000 C CNN
+F 2 "stepper_driver:STEPSTICK_TMC2209" H 5500 2800 60  0001 C CNN
+F 3 "" H 5600 3850 60  0001 C CNN
+F 4 "Digi-Key" H 5700 3000 60  0001 C CNN "Vendor"
+F 5 "ED90331-ND" H 5800 3100 60  0001 C CNN "Vendor Part Number"
+F 6 "CONN PIN RCPT .025-.037 SOLDER" H 5850 3100 60  0001 C CNN "Description"
+F 7 "16" H 6000 3300 60  0001 C CNN "Quantity"
+	1    5600 3850
+	1    0    0    -1
+$EndComp
+NoConn ~ 5500 3150
+NoConn ~ 5700 3150
+NoConn ~ 6200 3700
+NoConn ~ 6200 3800
+NoConn ~ 6200 3900
+NoConn ~ 6200 4000
+NoConn ~ 5650 4550
+NoConn ~ 5550 4550
+NoConn ~ 5000 4250
+NoConn ~ 5000 4150
+NoConn ~ 5000 4050
+NoConn ~ 5000 3950
+NoConn ~ 5000 3850
+NoConn ~ 5000 3750
+NoConn ~ 5000 3650
+NoConn ~ 5000 3550
+$Comp
+L stepper_driver:TERM_BLK_4_PIN_0.1_PITCH T1
+U 1 1 6172AC1B
+P 6900 3850
+F 0 "T1" H 6978 3892 50  0000 L CNN
+F 1 "TERM_BLK_4_PIN_0.1_PITCH" H 6978 3800 50  0000 L CNN
+F 2 "stepper_driver:TERM_BLK_4_PIN_0.1_PITCH" H 6800 4000 50  0001 C CNN
+F 3 "" H 6900 3850 50  0000 C CNN
+F 4 "Digi-Key" H 7000 4200 60  0001 C CNN "Vendor"
+F 5 "A98335-ND" H 7100 4300 60  0001 C CNN "Vendor Part Number"
+F 6 "TERM BLOCK 4POS SIDE ENT 2.54MM" H 7200 4400 60  0001 C CNN "Description"
+F 7 "TE Connectivity AMP Connectors" H 6900 3850 50  0001 C CNN "Manufacturer"
+F 8 "282834-4" H 6900 3850 50  0001 C CNN "Manufacturer Part Number"
+	1    6900 3850
+	1    0    0    -1
+$EndComp
+NoConn ~ 6700 3700
+NoConn ~ 6700 3800
+NoConn ~ 6700 3900
+NoConn ~ 6700 4000
 $EndSCHEMATC

Commit message: Add connectors
Parts:
- added T2: TERM_BLK_ANG_2_PIN_3.5MM_PITCH, stepper_driver:TERM_BLK_ANG_2_PIN_3.5MM_PITCH, symbol stepper_driver:TERM_BLK_ANG_2_PIN_3.5MM_PITCH
- added T3, T4: TERM_BLK_2_PIN_0.1_PITCH, stepper_driver:TERM_BLK_2_PIN_0.1_PITCH, symbol stepper_driver:TERM_BLK_2_PIN_0.1_PITCH
- SS1: Manufacturer (none) -> Mill-Max Manufacturing Corp.; Manufacturer Part Number (none) -> 0305-0-15-15-47-27-10-0
Connections:
- net labels added: A+, A-, B+, B-, DIR, GND, REF+, REF-, REFR+, REFR-, STEP, UART, VAA, VIO, VM
- wire segments 0 -> 23
- no-connect marks 24 -> 9
Changed lines of the file:
@@
 L stepper_driver:STEPSTICK_TMC2209 SS1
 U 1 1 6172192F
-P 5600 3850
-F 0 "SS1" H 5900 4400 60  0000 C CNN
-F 1 "STEPSTICK_TMC2209" H 6150 3300 60  0000 C CNN
-F 2 "stepper_driver:STEPSTICK_TMC2209" H 5500 2800 60  0001 C CNN
-F 3 "" H 5600 3850 60  0001 C CNN
-F 4 "Digi-Key" H 5700 3000 60  0001 C CNN "Vendor"
-F 5 "ED90331-ND" H 5800 3100 60  0001 C CNN "Vendor Part Number"
-F 6 "CONN PIN RCPT .025-.037 SOLDER" H 5850 3100 60  0001 C CNN "Description"
-F 7 "16" H 6000 3300 60  0001 C CNN "Quantity"
-	1    5600 3850
+P 5600 3650
+F 0 "SS1" H 5900 4200 60  0000 C CNN
+F 1 "STEPSTICK_TMC2209" H 6150 3100 60  0000 C CNN
+F 2 "stepper_driver:STEPSTICK_TMC2209" H 5500 2600 60  0001 C CNN
+F 3 "" H 5600 3650 60  0001 C CNN
+F 4 "Digi-Key" H 5700 2800 60  0001 C CNN "Vendor"
+F 5 "ED90331-ND" H 5800 2900 60  0001 C CNN "Vendor Part Number"
+F 6 "CONN PIN RCPT .025-.037 SOLDER" H 5850 2900 60  0001 C CNN "Description"
+F 7 "16" H 6000 3100 60  0001 C CNN "Quantity"
+F 8 "Mill-Max Manufacturing Corp." H 5600 3650 50  0001 C CNN "Manufacturer"
+F 9 "0305-0-15-15-47-27-10-0" H 5600 3650 50  0001 C CNN "Manufacturer Part Number"
+	1    5600 3650
 	1    0    0    -1
 $EndComp
-NoConn ~ 5500 3150
-NoConn ~ 5700 3150
-NoConn ~ 6200 3700
-NoConn ~ 6200 3800
-NoConn ~ 6200 3900
-NoConn ~ 6200 4000
-NoConn ~ 5650 4550
-NoConn ~ 5550 4550
-NoConn ~ 5000 4250
-NoConn ~ 5000 4150
 NoConn ~ 5000 4050
 NoConn ~ 5000 3950
 NoConn ~ 5000 3850
-NoConn ~ 5000 3750
 NoConn ~ 5000 3650
 NoConn ~ 5000 3550
@@
 L stepper_driver:TERM_BLK_4_PIN_0.1_PITCH T1
 U 1 1 6172AC1B
-P 6900 3850
-F 0 "T1" H 6978 3892 50  0000 L CNN
-F 1 "TERM_BLK_4_PIN_0.1_PITCH" H 6978 3800 50  0000 L CNN
-F 2 "stepper_driver:TERM_BLK_4_PIN_0.1_PITCH" H 6800 4000 50  0001 C CNN
-F 3 "" H 6900 3850 50  0000 C CNN
-F 4 "Digi-Key" H 7000 4200 60  0001 C CNN "Vendor"
-F 5 "A98335-ND" H 7100 4300 60  0001 C CNN "Vendor Part Number"
-F 6 "TERM BLOCK 4POS SIDE ENT 2.54MM" H 7200 4400 60  0001 C CNN "Description"
-F 7 "TE Connectivity AMP Connectors" H 6900 3850 50  0001 C CNN "Manufacturer"
-F 8 "282834-4" H 6900 3850 50  0001 C CNN "Manufacturer Part Number"
-	1    6900 3850
+P 7650 3650
+F 0 "T1" H 7728 3692 50  0000 L CNN
+F 1 "TERM_BLK_4_PIN_0.1_PITCH" H 7728 3600 50  0000 L CNN
+F 2 "stepper_driver:TERM_BLK_4_PIN_0.1_PITCH" H 7550 3800 50  0001 C CNN
+F 3 "" H 7650 3650 50  0000 C CNN
+F 4 "Digi-Key" H 7750 4000 60  0001 C CNN "Vendor"
+F 5 "A98335-ND" H 7850 4100 60  0001 C CNN "Vendor Part Number"
+F 6 "TERM BLOCK 4POS SIDE ENT 2.54MM" H 7950 4200 60  0001 C CNN "Description"
+F 7 "TE Connectivity AMP Connectors" H 7650 3650 50  0001 C CNN "Manufacturer"
+F 8 "282834-4" H 7650 3650 50  0001 C CNN "Manufacturer Part Number"
+	1    7650 3650
 	1    0    0    -1
 $EndComp
-NoConn ~ 6700 3700
-NoConn ~ 6700 3800
-NoConn ~ 6700 3900
-NoConn ~ 6700 4000
+Wire Wire Line
+	5000 3350 4900 3350
+Wire Wire Line
+	5000 3450 4900 3450
+Wire Wire Line
+	5000 3750 4900 3750
+Wire Wire Line
+	5500 2950 5500 2850
+Wire Wire Line
+	5700 2950 5700 2850
+Wire Wire Line
+	6200 3500 6300 3500
+Wire Wire Line
+	6200 3600 6300 3600
+Wire Wire Line
+	6200 3700 6300 3700
+Wire Wire Line
+	6200 3800 6300 3800
+Wire Wire Line
+	5550 4350 5550 4450
+Wire Wire Line
+	5650 4350 5650 4450
+Text Label 4900 3350 2    50   ~ 0
+STEP
+Text Label 4900 3450 2    50   ~ 0
+DIR
+Text Label 4900 3750 2    50   ~ 0
+UART
+Text Label 5500 2850 2    50   ~ 0
+VIO
+Text Label 5700 2850 2    50   ~ 0
+VM
+Text Label 6300 3500 0    50   ~ 0
+A+
+Text Label 6300 3600 0    50   ~ 0
+A-
+Text Label 6300 3700 0    50   ~ 0
+B+
+Text Label 6300 3800 0    50   ~ 0
+B-
+Wire Wire Line
+	5550 4450 5650 4450
+Wire Wire Line
+	5650 4450 5750 4450
+Connection ~ 5650 4450
+Text Label 5750 4450 0    50   ~ 0
+GND
+Wire Wire Line
+	7450 3800 7350 3800
+Wire Wire Line
+	7450 3700 7350 3700
+Wire Wire Line
+	7450 3600 7350 3600
+Wire Wire Line
+	7450 3500 7350 3500
+Text Label 7350 3700 2    50   ~ 0
+A+
+Text Label 7350 3800 2    50   ~ 0
+A-
+Text Label 7350 3600 2    50   ~ 0
+B+
+Text Label 7350 3500 2    50   ~ 0
+B-
+$Comp
+L stepper_driver:TERM_BLK_ANG_2_PIN_3.5MM_PITCH T2
+U 1 1 6178BDEE
+P 2500 2600
+F 0 "T2" H 2579 2642 50  0000 L CNN
+F 1 "TERM_BLK_ANG_2_PIN_3.5MM_PITCH" H 2579 2550 50  0000 L CNN
+F 2 "stepper_driver:TERM_BLK_ANG_2_PIN_3.5MM_PITCH" H 2400 2650 60  0001 C CNN
+F 3 "" H 2500 2600 60  0000 C CNN
+F 4 "Digi-Key" H 2600 2850 60  0001 C CNN "Vendor"
+F 5 "277-1779-ND" H 2700 2950 60  0001 C CNN "Vendor Part Number"
+F 6 "Phoenix Contact" H 2500 2600 50  0001 C CNN "Manufacturer"
+F 7 "1988956" H 2500 2600 50  0001 C CNN "Manufacturer Part Number"
+	1    2500 2600
+	1    0    0    -1
+$EndComp
+Wire Wire Line
+	2300 2550 2200 2550
+Wire Wire Line
+	2300 2650 2200 2650
+Text Label 2200 2550 2    50   ~ 0
+VAA
+Text Label 2200 2650 2    50   ~ 0
+GND
+$Comp
+L stepper_driver:TERM_BLK_2_PIN_0.1_PITCH T3
+U 1 1 61792CC9
+P 7650 4650
+F 0 "T3" H 7728 4692 50  0000 L CNN
+F 1 "TERM_BLK_2_PIN_0.1_PITCH" H 7728 4600 50  0000 L CNN
+F 2 "stepper_driver:TERM_BLK_2_PIN_0.1_PITCH" H 7550 4700 60  0001 C CNN
+F 3 "" H 7650 4650 60  0000 C CNN
+F 4 "Digi-Key" H 7750 4900 60  0001 C CNN "Vendor"
+F 5 "A98333-ND" H 7850 5000 60  0001 C CNN "Vendor Part Number"
+F 6 "TERM BLOCK 2POS SIDE ENT 2.54MM" H 7950 5100 60  0001 C CNN "Description"
+F 7 "TE Connectivity AMP Connectors" H 7650 4650 50  0001 C CNN "Manufacturer"
+F 8 "282834-2" H 7650 4650 50  0001 C CNN "Manufacturer Part Number"
+	1    7650 4650
+	1    0    0    -1
+$EndComp
+Wire Wire Line
+	7450 4600 7350 4600
+Wire Wire Line
+	7450 4700 7350 4700
+Text Label 7350 4600 2    50   ~ 0
+REF+
+Text Label 7350 4700 2    50   ~ 0
+REF-
+$Comp
+L stepper_driver:TERM_BLK_2_PIN_0.1_PITCH T4
+U 1 1 61794B89
+P 7650 4950
+F 0 "T4" H 7728 4992 50  0000 L CNN
+F 1 "TERM_BLK_2_PIN_0.1_PITCH" H 7728 4900 50  0000 L CNN
+F 2 "stepper_driver:TERM_BLK_2_PIN_0.1_PITCH" H 7550 5000 60  0001 C CNN
+F 3 "" H 7650 4950 60  0000 C CNN
+F 4 "Digi-Key" H 7750 5200 60  0001 C CNN "Vendor"
+F 5 "A98333-ND" H 7850 5300 60  0001 C CNN "Vendor Part Number"
+F 6 "TERM BLOCK 2POS SIDE ENT 2.54MM" H 7950 5400 60  0001 C CNN "Description"
+F 7 "TE Connectivity AMP Connectors" H 7650 4950 50  0001 C CNN "Manufacturer"
+F 8 "282834-2" H 7650 4950 50  0001 C CNN "Manufacturer Part Number"
+	1    7650 4950
+	1    0    0    -1
+$EndComp
+Wire Wire Line
+	7450 4900 7350 4900
+Wire Wire Line
+	7450 5000 7350 5000
+Text Label 7350 4900 2    50   ~ 0
+REFR+
+Text Label 7350 5000 2    50   ~ 0
+REFR-
 $EndSCHEMATC

Commit message: Add protection diodes
Parts:
- added C1: 100uF_POL, stepper_driver:CP_Elec_6.3x7.7_WURTH, symbol stepper_driver:100uF_POL
- added D1: DIODE_SCHOTTKY_45V_10A, stepper_driver:CFP15, symbol stepper_driver:DIODE_SCHOTTKY_45V_10A
- added D2: DIODE_TVS_ZENER_28V, stepper_driver:D_SMB_LITTELFUSE, symbol stepper_driver:DIODE_TVS_ZENER_28V
Connections:
- wire segments 23 -> 33

Commit message: Add power components
Parts:
- added C2, C3: 1uF, stepper_driver:SM0402, symbol stepper_driver:1uF_0402
- added C4, C5: 0.1uF, stepper_driver:SM0402, symbol stepper_driver:0.1uF_0402
- added R1, R2: 100, stepper_driver:SM0402, symbol stepper_driver:100_0402
- added REG1: CONV_DC_DC_3.3V_100MA, stepper_driver:SOT-23-3, symbol stepper_driver:CONV_DC_DC_3.3V_100MA
- added U1: SN65LVDM050QDRQ1, stepper_driver:SOIC_16_0.154IN, symbol stepper_driver:SN65LVDM050QDRQ1
- added U2: MAX6817, stepper_driver:MAX6817, symbol stepper_driver:MAX6817
Connections:
- net labels added: DIR_A, DIR_B, REF, REFR, REFR_A, REFR_B, REFR_D, REF_A, REF_B, REF_D, STEP_A, STEP_B, VCC, VDD
- net labels removed: REF+, REF-, REFR+, REFR-, VIO, VM
- wire segments 33 -> 72

Commit message: Add latched header
Parts:
- added P1: HEADER_02X05_LATCH, stepper_driver:HEADER_02x05_LATCH, symbol stepper_driver:HEADER_02X05_LATCH
Connections:
- wire segments 72 -> 84
Changed lines of the file:
@@
 	1100 1450 1000 1450
 Wire Wire Line
-	1100 1550 1000 1550
+	1100 1550 800  1550
 Text Label 1000 1450 2    50   ~ 0
 VAA
-Text Label 1000 1550 2    50   ~ 0
+Text Label 700  1550 2    50   ~ 0
 GND
 $Comp
 L stepper_driver:TERM_BLK_2_PIN_0.1_PITCH T3
 U 1 1 61792CC9
-P 7350 4550
-F 0 "T3" H 7428 4592 50  0000 L CNN
-F 1 "TERM_BLK_2_PIN_0.1_PITCH" H 7428 4500 50  0000 L CNN
-F 2 "stepper_driver:TERM_BLK_2_PIN_0.1_PITCH" H 7250 4600 60  0001 C CNN
-F 3 "" H 7350 4550 60  0000 C CNN
-F 4 "Digi-Key" H 7450 4800 60  0001 C CNN "Vendor"
-F 5 "A98333-ND" H 7550 4900 60  0001 C CNN "Vendor Part Number"
-F 6 "TERM BLOCK 2POS SIDE ENT 2.54MM" H 7650 5000 60  0001 C CNN "Description"
-F 7 "TE Connectivity AMP Connectors" H 7350 4550 50  0001 C CNN "Manufacturer"
-F 8 "282834-2" H 7350 4550 50  0001 C CNN "Manufacturer Part Number"
-	1    7350 4550
+P 7900 4850
+F 0 "T3" H 7978 4892 50  0000 L CNN
+F 1 "TERM_BLK_2_PIN_0.1_PITCH" H 7978 4800 50  0000 L CNN
+F 2 "stepper_driver:TERM_BLK_2_PIN_0.1_PITCH" H 7800 4900 60  0001 C CNN
+F 3 "" H 7900 4850 60  0000 C CNN
+F 4 "Digi-Key" H 8000 5100 60  0001 C CNN "Vendor"
+F 5 "A98333-ND" H 8100 5200 60  0001 C CNN "Vendor Part Number"
+F 6 "TERM BLOCK 2POS SIDE ENT 2.54MM" H 8200 5300 60  0001 C CNN "Description"
+F 7 "TE Connectivity AMP Connectors" H 7900 4850 50  0001 C CNN "Manufacturer"
+F 8 "282834-2" H 7900 4850 50  0001 C CNN "Manufacturer Part Number"
+	1    7900 4850
 	-1   0    0    1
 $EndComp
 Wire Wire Line
-	7550 4600 7650 4600
-Wire Wire Line
-	7550 4500 7650 4500
-Text Label 7650 4500 0    50   ~ 0
+	8100 4900 8200 4900
+Wire Wire Line
+	8100 4800 8200 4800
+Text Label 8200 4800 0    50   ~ 0
 REF
 $Comp
 L stepper_driver:TERM_BLK_2_PIN_0.1_PITCH T4
 U 1 1 61794B89
-P 7350 4850
-F 0 "T4" H 7428 4892 50  0000 L CNN
-F 1 "TERM_BLK_2_PIN_0.1_PITCH" H 7428 4800 50  0000 L CNN
-F 2 "stepper_driver:TERM_BLK_2_PIN_0.1_PITCH" H 7250 4900 60  0001 C CNN
-F 3 "" H 7350 4850 60  0000 C CNN
-F 4 "Digi-Key" H 7450 5100 60  0001 C CNN "Vendor"
-F 5 "A98333-ND" H 7550 5200 60  0001 C CNN "Vendor Part Number"
-F 6 "TERM BLOCK 2POS SIDE ENT 2.54MM" H 7650 5300 60  0001 C CNN "Description"
-F 7 "TE Connectivity AMP Connectors" H 7350 4850 50  0001 C CNN "Manufacturer"
-F 8 "282834-2" H 7350 4850 50  0001 C CNN "Manufacturer Part Number"
-	1    7350 4850
+P 7900 5150
+F 0 "T4" H 7978 5192 50  0000 L CNN
+F 1 "TERM_BLK_2_PIN_0.1_PITCH" H 7978 5100 50  0000 L CNN
+F 2 "stepper_driver:TERM_BLK_2_PIN_0.1_PITCH" H 7800 5200 60  0001 C CNN
+F 3 "" H 7900 5150 60  0000 C CNN
+F 4 "Digi-Key" H 8000 5400 60  0001 C CNN "Vendor"
+F 5 "A98333-ND" H 8100 5500 60  0001 C CNN "Vendor Part Number"
+F 6 "TERM BLOCK 2POS SIDE ENT 2.54MM" H 8200 5600 60  0001 C CNN "Description"
+F 7 "TE Connectivity AMP Connectors" H 7900 5150 50  0001 C CNN "Manufacturer"
+F 8 "282834-2" H 7900 5150 50  0001 C CNN "Manufacturer Part Number"
+	1    7900 5150
 	-1   0    0    1
 $EndComp
 Wire Wire Line
-	7550 4900 7650 4900
-Wire Wire Line
-	7550 4800 7650 4800
-Text Label 7650 4800 0    50   ~ 0
+	8100 5200 8200 5200
+Wire Wire Line
+	8100 5100 8200 5100
+Text Label 8200 5100 0    50   ~ 0
 REFR
 $Comp
@@
 L stepper_driver:0.1uF_0402 C5
 U 1 1 6180D67F
-P 8200 4650
-F 0 "C5" H 8250 4750 40  0000 L CNN
-F 1 "0.1uF" H 8200 4650 30  0000 C CNN
-F 2 "stepper_driver:SM0402" H 8238 4500 30  0001 C CNN
-F 3 "" H 8200 4650 60  0001 C CNN
-F 4 "Digi-Key" H 8300 4850 60  0001 C CNN "Vendor"
-F 5 "311-1375-1-ND" H 8400 4950 60  0001 C CNN "Vendor Part Number"
-F 6 "CAP CER 0.1UF 25V Y5V" H 8500 5050 60  0001 C CNN "Description"
-F 7 "0402" H 8200 4650 50  0001 C CNN "Package"
-F 8 "Yageo" H 8200 4650 50  0001 C CNN "Manufacturer"
-F 9 "CC0402ZRY5V8BB104" H 8200 4650 50  0001 C CNN "Manufacturer Part Number"
-	1    8200 4650
-	1    0    0    -1
-$EndComp
-Wire Wire Line
-	8200 4450 8200 4350
-Text Label 8200 4350 0    50   ~ 0
+P 8750 4950
+F 0 "C5" H 8800 5050 40  0000 L CNN
+F 1 "0.1uF" H 8750 4950 30  0000 C CNN
+F 2 "stepper_driver:SM0402" H 8788 4800 30  0001 C CNN
+F 3 "" H 8750 4950 60  0001 C CNN
+F 4 "Digi-Key" H 8850 5150 60  0001 C CNN "Vendor"
+F 5 "311-1375-1-ND" H 8950 5250 60  0001 C CNN "Vendor Part Number"
+F 6 "CAP CER 0.1UF 25V Y5V" H 9050 5350 60  0001 C CNN "Description"
+F 7 "0402" H 8750 4950 50  0001 C CNN "Package"
+F 8 "Yageo" H 8750 4950 50  0001 C CNN "Manufacturer"
+F 9 "CC0402ZRY5V8BB104" H 8750 4950 50  0001 C CNN "Manufacturer Part Number"
+	1    8750 4950
+	1    0    0    -1
+$EndComp
+Wire Wire Line
+	8750 4750 8750 4650
+Text Label 8750 4650 0    50   ~ 0
 VDD
 Wire Wire Line
-	8200 4850 8200 4950
-Text Label 8200 4950 0    50   ~ 0
+	8750 5150 8750 5250
+Text Label 8750 5250 0    50   ~ 0
 GND
 $Comp
 L stepper_driver:MAX6817 U2
 U 1 1 61814C7C
-P 9250 4650
-F 0 "U2" H 9450 4900 60  0000 C CNN
-F 1 "MAX6817" H 9500 4400 60  0000 C CNN
-F 2 "stepper_driver:MAX6817" H 9250 3900 60  0001 C CNN
-F 3 "" H 9250 4650 60  0000 C CNN
-F 4 "IC DEBOUNCER SWITCH DUAL" H 9250 4000 60  0001 C CNN "Description"
-F 5 "SOT-23-6" H 9250 4650 60  0001 C CNN "Package"
-F 6 "Maxim Integrated" H 9250 4650 60  0001 C CNN "Manufacturer"
-F 7 "MAX6817EUT+T" H 9250 4650 60  0001 C CNN "Manufacturer Part Number"
-F 8 "Mouser" H 9250 3700 60  0001 C CNN "Vendor"
-F 9 "MAX6817EUT+T" H 9250 3800 60  0001 C CNN "Vendor Part Number"
-	1    9250 4650
-	1    0    0    -1
-$EndComp
-Text Label 7650 4600 0    50   ~ 0
-GND
-Text Label 7650 4900 0    50   ~ 0
-GND
-Wire Wire Line
-	9250 4350 9250 4250
-Wire Wire Line
-	9250 4950 9250 5050
-Wire Wire Line
-	9650 4700 9750 4700
-Wire Wire Line
-	9650 4800 9750 4800
-Wire Wire Line
-	8850 4700 8750 4700
-Wire Wire Line
-	8850 4800 8750 4800
-Text Label 8750 4700 2    50   ~ 0
+P 9800 4950
+F 0 "U2" H 10000 5200 60  0000 C CNN
+F 1 "MAX6817" H 10050 4700 60  0000 C CNN
+F 2 "stepper_driver:MAX6817" H 9800 4200 60  0001 C CNN
+F 3 "" H 9800 4950 60  0000 C CNN
+F 4 "IC DEBOUNCER SWITCH DUAL" H 9800 4300 60  0001 C CNN "Description"
+F 5 "SOT-23-6" H 9800 4950 60  0001 C CNN "Package"
+F 6 "Maxim Integrated" H 9800 4950 60  0001 C CNN "Manufacturer"
+F 7 "MAX6817EUT+T" H 9800 4950 60  0001 C CNN "Manufacturer Part Number"
+F 8 "Mouser" H 9800 4000 60  0001 C CNN "Vendor"
+F 9 "MAX6817EUT+T" H 9800 4100 60  0001 C CNN "Vendor Part Number"
+	1    9800 4950
+	1    0    0    -1
+$EndComp
+Text Label 8200 4900 0    50   ~ 0
+GND
+Text Label 8200 5200 0    50   ~ 0
+GND
+Wire Wire Line
+	9800 4650 9800 4550
+Wire Wire Line
+	9800 5250 9800 5350
+Wire Wire Line
+	10200 5000 10300 5000
+Wire Wire Line
+	10200 5100 10300 5100
+Wire Wire Line
+	9400 5000 9300 5000
+Wire Wire Line
+	9400 5100 9300 5100
+Text Label 9300 5000 2    50   ~ 0
 REF
-Text Label 8750 4800 2    50   ~ 0
+Text Label 9300 5100 2    50   ~ 0
 REFR
-Text Label 9750 4800 0    50   ~ 0
+Text Label 10300 5100 0    50   ~ 0
 REFR_D
-Text Label 9750 4700 0    50   ~ 0
+Text Label 10300 5000 0    50   ~ 0
 REF_D
-Text Label 9250 4250 0    50   ~ 0
+Text Label 9800 4550 0    50   ~ 0
 VDD
-Text Label 9250 5050 0    50   ~ 0
+Text Label 9800 5350 0    50   ~ 0
 GND
 Text Label 2600 4400 2    50   ~ 0
@@
 Text Label 3600 4550 0    50   ~ 0
 REFR_B
+$Comp
+L stepper_driver:HEADER_02X05_LATCH P1
+U 1 1 617CC4ED
+P 5950 5000
+F 0 "P1" H 5950 5300 50  0000 C CNN
+F 1 "HEADER_02X05_LATCH" H 5950 4700 50  0000 C CNN
+F 2 "stepper_driver:HEADER_02x05_LATCH" H 5950 3800 60  0001 C CNN
+F 3 "" H 5950 3800 60  0000 C CNN
+F 4 "Digi-Key" H 6050 5400 60  0001 C CNN "Vendor"
+F 5 "MHS10N-ND" H 6150 5500 60  0001 C CNN "Vendor Part Number"
+F 6 "CONN HEADER VERT 10POS 2.54MM" H 6250 5600 60  0001 C CNN "Description"
+F 7 "3M" H 5950 5000 50  0001 C CNN "Manufacturer"
+F 8 "N3793-6302RB" H 5950 5000 50  0001 C CNN "Manufacturer Part Number"
+	1    5950 5000
+	1    0    0    -1
+$EndComp
+Wire Wire Line
+	5700 4800 5600 4800
+Wire Wire Line
+	5700 4900 5600 4900
+Text Label 5600 4900 2    50   ~ 0
+DIR_A
+Text Label 5600 4800 2    50   ~ 0
+STEP_A
+Wire Wire Line
+	6200 4800 6300 4800
+Text Label 6300 4800 0    50   ~ 0
+STEP_B
+Wire Wire Line
+	6200 4900 6300 4900
+Text Label 6300 4900 0    50   ~ 0
+DIR_B
+Wire Wire Line
+	5700 5000 5600 5000
+Text Label 5600 5000 2    50   ~ 0
+UART
+Wire Wire Line
+	6200 5000 6300 5000
+Text Label 6300 5000 0    50   ~ 0
+GND
+Wire Wire Line
+	5700 5100 5600 5100
+Text Label 5600 5100 2    50   ~ 0
+REF_A
+Wire Wire Line
+	5700 5200 5600 5200
+Text Label 5600 5200 2    50   ~ 0
+REFR_A
+Wire Wire Line
+	6200 5200 6300 5200
+Text Label 6300 5200 0    50   ~ 0
+REFR_B
+Wire Wire Line
+	6200 5100 6300 5100
+Text Label 6300 5100 0    50   ~ 0
+REF_B
+$Comp
+L user_power:PWR_FLAG #FLG0101
+U 1 1 617E32B0
+P 800 1400
+F 0 "#FLG0101" H 800 1475 50  0001 C CNN
+F 1 "PWR_FLAG" H 800 1575 50  0000 C CNN
+F 2 "" H 800 1400 50  0001 C CNN
+F 3 "~" H 800 1400 50  0001 C CNN
+	1    800  1400
+	1    0    0    -1
+$EndComp
+Wire Wire Line
+	800  1400 800  1550
+Connection ~ 800  1550
+Wire Wire Line
+	800  1550 700  1550
 $EndSCHEMATC
