File: stepper_driver.kicad_pcb (KiCad board)
At the start: 2 copper layers, 203.2 x 147.3 mm, 189 parts, among them P1 PWR_JACK_2.5x5.5_SMD_VERT, P10 RECEPTACLE_2MM, P11 RECEPTACLE_2MM, P12 RECEPTACLE_2MM, P13 RECEPTACLE_2MM, P14 RECEPTACLE_2MM, P2 BNC, P3 RECEPTACLE_2MM, P4 RECEPTACLE_2MM, P5 RECEPTACLE_2MM, P6 RECEPTACLE_2MM, P7 RECEPTACLE_2MM, P8 RECEPTACLE_2MM, P9 RECEPTACLE_2MM, T1 TERM_BLK_ANG_2_PIN_3.5MM_PITCH, T10 TERM_BLK_ANG_2_PIN_3.5MM_PITCH, T11 TERM_BLK_ANG_2_PIN_3.5MM_PITCH, T12 TERM_BLK_ANG_2_PIN_3.5MM_PITCH, T2 TERM_BLK_ANG_2_PIN_3.5MM_PITCH, T3 TERM_BLK_ANG_2_PIN_3.5MM_PITCH, T4 TERM_BLK_ANG_2_PIN_3.5MM_PITCH, T5 TERM_BLK_ANG_2_PIN_3.5MM_PITCH, T6 TERM_BLK_ANG_2_PIN_3.5MM_PITCH, T7 TERM_BLK_ANG_2_PIN_3.5MM_PITCH, T8 TERM_BLK_ANG_2_PIN_3.5MM_PITCH, T9 TERM_BLK_ANG_2_PIN_3.5MM_PITCH, U1 AT42QT2120-MMHR, U10 DRV103, U11 DRV103, U12 DRV103, U13 DRV103, U2 DRV103, U3 DRV103, U4 DRV103, U5 DRV103, U6 DRV103, U7 DRV103, U8 DRV103, U9 DRV103

Commit message: Clear schematic and board
Parts:
- removed C1: 10uF, stepper_driver:SM0805
- removed C10, C12, C14, C16, C18, C20, C22, C24, C26, C4, C6, C8: 1uF, lickport_interface:SM0402_POL
- removed C11, C13, C15, C17, C19, C21, C23, C25, C27, C5, C7, C9: 47nF, lickport_interface:SM0402
- removed C2: 1uF, stepper_driver:SM0402_POL
- removed C3: 0.1uF, lickport_interface:SM0402
- removed D1: DIODE_SCHOTTKY_45V_10A, stepper_driver:CFP15
- removed D10, D12, D14, D16, D18, D20, D22, D24, D26, D4, D6, D8: DIODE_LOW_REV_CURRENT_0402, lickport_interface:SM0402_POL
- removed D11, D13, D15, D17, D19, D21, D23, D25, D3, D5, D7, D9: DIODE_SCHOTTKY_0402, lickport_interface:SM0402_POL
- removed D2: DIODE_LOW_REV_CURRENT_0402, stepper_driver:SM0402_POL
- removed FID1, FID2, FID3, FID4: FIDUCIAL, stepper_driver:FIDUCIAL
- removed L1: LED_GRN, stepper_driver:LED0805
- removed L10, L11, L12, L13, L2, L3, L4, L5, L6, L7, L8, L9: LED_GRN, lickport_interface:LED0805
- removed MH1, MH10, MH11, MH12, MH13, MH14, MH2, MH3, MH4, MH5, MH6, MH7, MH8, MH9: MOUNTING_HOLE_4-40, stepper_driver:MOUNTING_HOLE_4-40
- removed P1: PWR_JACK_2.5x5.5_SMD_VERT, stepper_driver:DCJACK_3PIN_SMD_VERT
- removed P10, P11, P12, P13, P14, P3, P4, P5, P6, P7, P8, P9: RECEPTACLE_2MM, lickport_interface:RECEPTACLE_2MM
- removed P2: BNC, stepper_driver:BNC
- removed R1, R2, R3: 2.2k, stepper_driver:SM0402
- removed R10, R14, R18, R22, R26, R30, R34, R38, R42, R46, R50, R6: 137k, lickport_interface:SM0402
- removed R11, R15, R19, R23, R27, R31, R35, R39, R43, R47, R51, R7: 205k, lickport_interface:SM0402
- removed R12, R16, R20, R24, R28, R32, R36, R40, R44, R48, R52, R8: 2.2k, lickport_interface:SM0402
- removed R13, R17, R21, R25, R29, R33, R37, R41, R45, R49, R53, R9: 20k, lickport_interface:SM0402
- removed R4, R5: 47k, stepper_driver:SM0402
- removed S1, S10, S11, S12, S2, S3, S4, S5, S6, S7, S8, S9: CLIPPARD-NPV2-1C-23-24, lickport_interface:CLIPPARD_NPV2-1C-23-24
- removed T1, T10, T11, T12, T2, T3, T4, T5, T6, T7, T8, T9: TERM_BLK_ANG_2_PIN_3.5MM_PITCH, lickport_interface:TERM_BLK_ANG_2_PIN_3.5MM_PITCH
- removed TEENSY1: TEENSY_4.0_HEADERS, stepper_driver:TEENSY_4.0_HEADERS
- removed U1: AT42QT2120-MMHR, stepper_driver:QFN-20-1EP_3x3mm_P0.45mm_EP1.6x1.6mm
- removed U10, U11, U12, U13, U2, U3, U4, U5, U6, U7, U8, U9: DRV103, lickport_interface:SOIC_8
Routing:
- net GND: track 931.1 -> 0.00 mm, vias 2 -> 0
- net VCC: track 869.5 -> 0.00 mm
- net /lickport_interface_6/SENSE: track 157.7 -> 0.00 mm
- net /SOLENOID_4: track 152.0 -> 0.00 mm, vias 1 -> 0
- net /SOLENOID_1: track 146.5 -> 0.00 mm, vias 1 -> 0
- net /lickport_interface_10/SENSE: track 146.5 -> 0.00 mm
- net /SOLENOID_3: track 141.1 -> 0.00 mm, vias 1 -> 0
- net /SYNC: track 126.3 -> 0.00 mm, vias 1 -> 0
- net /lickport_interface_8/SENSE: track 123.8 -> 0.00 mm
- net /lickport_interface_5/SENSE: track 123.5 -> 0.00 mm
- net /lickport_interface_4/SENSE: track 123.2 -> 0.00 mm
- net /lickport_interface_1/SENSE: track 122.6 -> 0.00 mm
- net /lickport_interface_2/SENSE: track 122.2 -> 0.00 mm
- net /SOLENOID_0: track 121.5 -> 0.00 mm, vias 2 -> 0
- net /SOLENOID_10: track 112.5 -> 0.00 mm
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- removed copper zone on B.Cu, net GND
- removed copper zone on F.Cu, net GND
Other:
- board outline removed
- board text removed: "0"
- board text removed: "1"
- board text removed: "10"
- board text removed: "11"
- board text removed: "2"
- board text removed: "2.5x5.5 Center + +24VDC"
- board text removed: "3"
- board text removed: "4"
- board text removed: "5"
- board text removed: "6"
- board text removed: "7"
- board text removed: "8"
- board text removed: "9"
- board text removed: "POWER"
- board text removed: "SYNC"
- board text removed: "stepper_driver Janelia Research Campus 06/2021 ver 1.1"

Commit message: Add mounting holes, stepstick, and term block
Parts:
- added FID1: FIDUCIAL, stepper_driver:FIDUCIAL, F.Cu at (121.9, 71.1)
- added FID2: FIDUCIAL, stepper_driver:FIDUCIAL, F.Cu at (157.5, 71.1)
- added FID3: FIDUCIAL, stepper_driver:FIDUCIAL, F.Cu at (157.5, 106.7)
- added FID4: FIDUCIAL, stepper_driver:FIDUCIAL, F.Cu at (121.9, 106.7)
- added MH1: MOUNTING_HOLE_4-40, stepper_driver:MOUNTING_HOLE_4-40, F.Cu at (124.2, 73.4)
- added MH2: MOUNTING_HOLE_4-40, stepper_driver:MOUNTING_HOLE_4-40, F.Cu at (155.2, 73.4)
- added MH3: MOUNTING_HOLE_4-40, stepper_driver:MOUNTING_HOLE_4-40, F.Cu at (155.2, 104.4)
- added MH4: MOUNTING_HOLE_4-40, stepper_driver:MOUNTING_HOLE_4-40, F.Cu at (124.2, 104.4)
- added SS1: STEPSTICK_TMC2209, stepper_driver:STEPSTICK_TMC2209, F.Cu at (139.7, 83.8)
- added T1: TERM_BLK_4_PIN_0.1_PITCH, stepper_driver:TERM_BLK_4_PIN_0.1_PITCH, F.Cu at (139.7, 71.1)
Other:
- board outline added: 41.9 x 41.9 mm

Commit message: Add connectors
Parts:
- added T2: TERM_BLK_ANG_2_PIN_3.5MM_PITCH, stepper_driver:TERM_BLK_ANG_2_PIN_3.5MM_PITCH, F.Cu at (123.2, 83.8)
- added T3: TERM_BLK_2_PIN_0.1_PITCH, stepper_driver:TERM_BLK_2_PIN_0.1_PITCH, F.Cu at (156.6, 86.8)
- added T4: TERM_BLK_2_PIN_0.1_PITCH, stepper_driver:TERM_BLK_2_PIN_0.1_PITCH, F.Cu at (156.6, 93.7)
Connections:
- SS1 pad 1: (no net) -> /GND
- SS1 pad 3: (no net) -> /A-
- SS1 pad 4: (no net) -> /A+
- SS1 pad 5: (no net) -> /B+
- SS1 pad 6: (no net) -> /B-
- SS1 pad 7: (no net) -> /GND
- T1 pad 1: (no net) -> /B-
- T1 pad 2: (no net) -> /B+
- T1 pad 3: (no net) -> /A+
- T1 pad 4: (no net) -> /A-
Changed lines of the file:
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@@
     (tracks 0)
     (zones 0)
-    (modules 10)
-    (nets 1)
+    (modules 13)
+    (nets 6)
   )
   (page A4)
@@
   )
   (net 0 "")
+  (net 1 /GND)
+  (net 2 /A-)
+  (net 3 /A+)
+  (net 4 /B+)
+  (net 5 /B-)
   (net_class Default "This is the default net class."
     (clearance 0.1016)
@@
     (diff_pair_width 0.254)
     (diff_pair_gap 0.254)
+    (add_net /A+)
+    (add_net /A-)
+    (add_net /B+)
+    (add_net /B-)
+    (add_net /GND)
   )
   (net_class POWER ""
@@
       (effects (font (size 0.254 0.254) (thickness 0.0635)))
     )
+    (fp_circle (center 0 0) (end 0.75 0) (layer F.CrtYd) (width 0.05))
     (fp_circle (center 0 0) (end 0.5 0) (layer F.Fab) (width 0.1))
-    (fp_circle (center 0 0) (end 0.75 0) (layer F.CrtYd) (width 0.05))
     (fp_text user %R (at 0 0) (layer F.Fab)
       (effects (font (size 0.2 0.2) (thickness 0.04)))
@@
       (effects (font (size 0.254 0.254) (thickness 0.0635)))
     )
+    (fp_circle (center 0 0) (end 0.5 0) (layer F.Fab) (width 0.1))
+    (fp_circle (center 0 0) (end 0.75 0) (layer F.CrtYd) (width 0.05))
     (fp_text user %R (at 0 0) (layer F.Fab)
       (effects (font (size 0.2 0.2) (thickness 0.04)))
     )
-    (fp_circle (center 0 0) (end 0.75 0) (layer F.CrtYd) (width 0.05))
-    (fp_circle (center 0 0) (end 0.5 0) (layer F.Fab) (width 0.1))
     (pad ~ smd circle (at 0 0) (size 0.5 0.5) (layers F.Cu F.Mask)
       (solder_mask_margin 0.25) (clearance 0.25))
@@
       (effects (font (size 0.254 0.254) (thickness 0.0635)))
     )
+    (fp_circle (center 0 0) (end 0.75 0) (layer F.CrtYd) (width 0.05))
     (fp_circle (center 0 0) (end 0.5 0) (layer F.Fab) (width 0.1))
-    (fp_circle (center 0 0) (end 0.75 0) (layer F.CrtYd) (width 0.05))
     (fp_text user %R (at 0 0) (layer F.Fab)
       (effects (font (size 0.2 0.2) (thickness 0.04)))
@@
       (effects (font (size 0.254 0.254) (thickness 0.0635)))
     )
+    (fp_circle (center 0 0) (end 0.5 0) (layer F.Fab) (width 0.1))
+    (fp_circle (center 0 0) (end 0.75 0) (layer F.CrtYd) (width 0.05))
     (fp_text user %R (at 0 0) (layer F.Fab)
       (effects (font (size 0.2 0.2) (thickness 0.04)))
     )
-    (fp_circle (center 0 0) (end 0.75 0) (layer F.CrtYd) (width 0.05))
-    (fp_circle (center 0 0) (end 0.5 0) (layer F.Fab) (width 0.1))
     (pad ~ smd circle (at 0 0) (size 0.5 0.5) (layers F.Cu F.Mask)
       (solder_mask_margin 0.25) (clearance 0.25))
@@
       (effects (font (size 1.016 1.016) (thickness 0.254)))
     )
+    (fp_line (start -7.62 -10.16) (end -7.62 10.16) (layer F.SilkS) (width 0.2286))
+    (fp_line (start -7.62 10.16) (end 7.62 10.16) (layer F.SilkS) (width 0.2286))
+    (fp_line (start 7.62 10.16) (end 7.62 -10.16) (layer F.SilkS) (width 0.2286))
     (fp_line (start 7.62 -10.16) (end -7.62 -10.16) (layer F.SilkS) (width 0.2286))
-    (fp_line (start 7.62 10.16) (end 7.62 -10.16) (layer F.SilkS) (width 0.2286))
-    (fp_line (start -7.62 10.16) (end 7.62 10.16) (layer F.SilkS) (width 0.2286))
-    (fp_line (start -7.62 -10.16) (end -7.62 10.16) (layer F.SilkS) (width 0.2286))
     (fp_text user DIR (at 2.54 -8.89 90) (layer F.SilkS)
       (effects (font (size 1.016 1.016) (thickness 0.254)))
@@
       (effects (font (size 1.016 1.016) (thickness 0.254)))
     )
-    (pad 1 thru_hole rect (at -6.35 -8.89 270) (size 3.048 2.032) (drill 1.5494) (layers *.Cu *.Mask))
+    (pad 1 thru_hole rect (at -6.35 -8.89 270) (size 3.048 2.032) (drill 1.5494) (layers *.Cu *.Mask)
+      (net 1 /GND))
     (pad 2 thru_hole oval (at -6.35 -6.35 270) (size 3.048 2.032) (drill 1.5494) (layers *.Cu *.Mask))
-    (pad 3 thru_hole oval (at -6.35 -3.81 270) (size 3.048 2.032) (drill 1.5494) (layers *.Cu *.Mask))
-    (pad 4 thru_hole oval (at -6.35 -1.27 270) (size 3.048 2.032) (drill 1.5494) (layers *.Cu *.Mask))
-    (pad 5 thru_hole oval (at -6.35 1.27 270) (size 3.048 2.032) (drill 1.5494) (layers *.Cu *.Mask))
-    (pad 6 thru_hole oval (at -6.35 3.81 270) (size 3.048 2.032) (drill 1.5494) (layers *.Cu *.Mask))
-    (pad 7 thru_hole oval (at -6.35 6.35 270) (size 3.048 2.032) (drill 1.5494) (layers *.Cu *.Mask))
+    (pad 3 thru_hole oval (at -6.35 -3.81 270) (size 3.048 2.032) (drill 1.5494) (layers *.Cu *.Mask)
+      (net 2 /A-))
+    (pad 4 thru_hole oval (at -6.35 -1.27 270) (size 3.048 2.032) (drill 1.5494) (layers *.Cu *.Mask)
+      (net 3 /A+))
+    (pad 5 thru_hole oval (at -6.35 1.27 270) (size 3.048 2.032) (drill 1.5494) (layers *.Cu *.Mask)
+      (net 4 /B+))
+    (pad 6 thru_hole oval (at -6.35 3.81 270) (size 3.048 2.032) (drill 1.5494) (layers *.Cu *.Mask)
+      (net 5 /B-))
+    (pad 7 thru_hole oval (at -6.35 6.35 270) (size 3.048 2.032) (drill 1.5494) (layers *.Cu *.Mask)
+      (net 1 /GND))
     (pad 8 thru_hole oval (at -6.35 8.89 270) (size 3.048 2.032) (drill 1.5494) (layers *.Cu *.Mask))
     (pad 16 thru_hole oval (at 6.35 8.89 270) (size 3.048 2.032) (drill 1.5494) (layers *.Cu *.Mask))
@@
       (effects (font (size 0.762 0.762) (thickness 0.1905)))
     )
+    (fp_line (start -5.31 -3.25) (end -5.31 3.25) (layer F.SilkS) (width 0.25))
+    (fp_line (start -5.31 3.25) (end 5.31 3.25) (layer F.SilkS) (width 0.25))
+    (fp_line (start 5.31 -3.25) (end 5.31 3.25) (layer F.SilkS) (width 0.25))
     (fp_line (start -5.31 -3.25) (end 5.31 -3.25) (layer F.SilkS) (width 0.25))
-    (fp_line (start 5.31 -3.25) (end 5.31 3.25) (layer F.SilkS) (width 0.25))
-    (fp_line (start -5.31 3.25) (end 5.31 3.25) (layer F.SilkS) (width 0.25))
-    (fp_line (start -5.31 -3.25) (end -5.31 3.25) (layer F.SilkS) (width 0.25))
-    (pad 1 thru_hole rect (at -3.81 0) (size 2 2.54) (drill 1.1) (layers *.Cu *.Mask))
-    (pad 2 thru_hole oval (at -1.27 0) (size 2 2.54) (drill 1.1) (layers *.Cu *.Mask))
-    (pad 3 thru_hole oval (at 1.27 0) (size 2 2.54) (drill 1.1) (layers *.Cu *.Mask))
-    (pad 4 thru_hole oval (at 3.81 0) (size 2 2.54) (drill 1.1) (layers *.Cu *.Mask))
+    (pad 1 thru_hole rect (at -3.81 0) (size 2 2.54) (drill 1.1) (layers *.Cu *.Mask)
+      (net 5 /B-))
+    (pad 2 thru_hole oval (at -1.27 0) (size 2 2.54) (drill 1.1) (layers *.Cu *.Mask)
+      (net 4 /B+))
+    (pad 3 thru_hole oval (at 1.27 0) (size 2 2.54) (drill 1.1) (layers *.Cu *.Mask)
+      (net 3 /A+))
+    (pad 4 thru_hole oval (at 3.81 0) (size 2 2.54) (drill 1.1) (layers *.Cu *.Mask)
+      (net 2 /A-))
+  )
+  (module stepper_driver:TERM_BLK_ANG_2_PIN_3.5MM_PITCH (layer F.Cu)
+    (at 123.19 83.82 180)
+    (fp_text reference T2 (at 0 -9.652) (layer F.SilkS)
+      (effects (font (size 1.016 1.016) (thickness 0.254)))
+    )
+    (fp_text value TERM_BLK_ANG_2_PIN_3.5MM_PITCH (at 0 3.175 180) (layer F.SilkS) hide
+      (effects (font (size 0.508 0.508) (thickness 0.127)))
+    )
+    (fp_line (start -1.75 -7.5) (end -2.25 -8.5) (layer F.SilkS) (width 0.2794))
+    (fp_line (start -1.25 -8.5) (end -1.75 -7.5) (layer F.SilkS) (width 0.2794))
+    (fp_line (start -2.25 -8.5) (end -1.25 -8.5) (layer F.SilkS) (width 0.2794))
+    (fp_line (start -3.5 -8.8) (end 3.5 -8.8) (layer F.SilkS) (width 0.3))
+    (fp_line (start 3.5 -8.8) (end 3.5 2.4) (layer F.SilkS) (width 0.3))
+    (fp_line (start -3.5 2.4) (end 3.5 2.4) (layer F.SilkS) (width 0.3))
+    (fp_line (start -3.5 -8.8) (end -3.5 2.4) (layer F.SilkS) (width 0.3))
+    (pad 1 thru_hole rect (at -1.75 0 180) (size 2.5 3.5) (drill 1.3) (layers *.Cu *.Mask))
+    (pad 2 thru_hole oval (at 1.75 0 180) (size 2.5 3.5) (drill 1.3) (layers *.Cu *.Mask)
+      (net 1 /GND))
+  )
+  (module stepper_driver:TERM_BLK_2_PIN_0.1_PITCH (layer F.Cu)
+    (at 156.578299 86.779101 270)
+    (fp_text reference T3 (at 0 -4.445 90) (layer F.SilkS)
+      (effects (font (size 1.016 1.016) (thickness 0.254)))
+    )
+    (fp_text value TERM_BLK_2_PIN_0.1_PITCH (at 0 4.445 270) (layer F.SilkS)
+      (effects (font (size 0.762 0.762) (thickness 0.1905)))
+    )
+    (fp_line (start -2.7686 -3.2512) (end 2.7686 -3.2512) (layer F.SilkS) (width 0.381))
+    (fp_line (start 2.7686 -3.2512) (end 2.7686 3.2512) (layer F.SilkS) (width 0.381))
+    (fp_line (start -2.7686 3.2512) (end 2.7686 3.2512) (layer F.SilkS) (width 0.381))
+    (fp_line (start -2.7686 -3.2512) (end -2.7686 3.2512) (layer F.SilkS) (width 0.381))
+    (pad 1 thru_hole rect (at -1.27 0 270) (size 1.905 2.54) (drill 1.1176) (layers *.Cu *.Mask))
+    (pad 2 thru_hole oval (at 1.27 0 270) (size 1.905 2.54) (drill 1.4224) (layers *.Cu *.Mask))
+  )
+  (module stepper_driver:TERM_BLK_2_PIN_0.1_PITCH (layer F.Cu)
+    (at 156.578299 93.689101 270)
+    (fp_text reference T4 (at 0 -4.445 90) (layer F.SilkS)
+      (effects (font (size 1.016 1.016) (thickness 0.254)))
+    )
+    (fp_text value TERM_BLK_2_PIN_0.1_PITCH (at 0 4.445 270) (layer F.SilkS)
+      (effects (font (size 0.762 0.762) (thickness 0.1905)))
+    )
+    (fp_line (start -2.7686 -3.2512) (end -2.7686 3.2512) (layer F.SilkS) (width 0.381))
+    (fp_line (start -2.7686 3.2512) (end 2.7686 3.2512) (layer F.SilkS) (width 0.381))
+    (fp_line (start 2.7686 -3.2512) (end 2.7686 3.2512) (layer F.SilkS) (width 0.381))
+    (fp_line (start -2.7686 -3.2512) (end 2.7686 -3.2512) (layer F.SilkS) (width 0.381))
+    (pad 2 thru_hole oval (at 1.27 0 270) (size 1.905 2.54) (drill 1.4224) (layers *.Cu *.Mask))
+    (pad 1 thru_hole rect (at -1.27 0 270) (size 1.905 2.54) (drill 1.1176) (layers *.Cu *.Mask))
   )
   (gr_arc (start 121.92 106.68) (end 118.745 106.68) (angle -90) (layer Edge.Cuts) (width 0.2286))
