File: stepper_driver/assembly.kicad_sch (KiCad schematic)
At the start: 8 parts

Commit message: Initial 2.0 schematic layout
Other:
- company: (none) -> Howard Hughes Medical Institute
- title: (none) -> stepper_driver
Changed lines of the file:
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@@
 (kicad_sch (version 20230121) (generator eeschema)
   (paper "A4")
+  (title_block
+    (title "stepper_driver")
+    (date "2023-03-31")
+    (rev "2.0")
+    (company "Howard Hughes Medical Institute")
+  )
   (wire (pts (xy 147.32 106.68) (xy 147.32 109.22))
     (stroke (width 0) (type default))
