File: stepper_driver/assembly.kicad_sch (KiCad schematic)
At the start: 8 parts

Commit message: Fix pcb issues
Changed lines of the file:
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@@
   (symbol (lib_id "Janelia:MOUNTING_HOLE_3") (at 135.89 106.68 0) (unit 1)
     (in_bom no) (on_board yes) (dnp no) (fields_autoplaced)
-    (property "Reference" "H1" (at 138.43 104.013 0)
+    (property "Reference" "H1" (at 138.43 103.378 0)
       (effects (font (size 1.27 1.27)) (justify left))
     )
@@
   (symbol (lib_id "Janelia:MOUNTING_HOLE_3") (at 146.05 106.68 0) (unit 1)
     (in_bom no) (on_board yes) (dnp no) (fields_autoplaced)
-    (property "Reference" "H2" (at 148.59 104.013 0)
+    (property "Reference" "H2" (at 148.59 103.378 0)
       (effects (font (size 1.27 1.27)) (justify left))
     )
@@
   (symbol (lib_id "Janelia:MOUNTING_HOLE_3") (at 156.21 106.68 0) (unit 1)
     (in_bom no) (on_board yes) (dnp no) (fields_autoplaced)
-    (property "Reference" "H3" (at 158.75 104.013 0)
+    (property "Reference" "H3" (at 158.75 103.378 0)
       (effects (font (size 1.27 1.27)) (justify left))
     )
@@
   (symbol (lib_id "Janelia:MOUNTING_HOLE_3") (at 166.37 106.68 0) (unit 1)
     (in_bom no) (on_board yes) (dnp no) (fields_autoplaced)
-    (property "Reference" "H4" (at 168.91 104.013 0)
-      (effects (font (size 1.27 1.27)) (justify left))
-    )
+    (property "Reference" "H4" (at 168.91 103.378 0)
+      (effects (font (size 1.27 1.27)) (justify left))
+    )
