File: stepper_driver/connectors.kicad_sch (KiCad schematic)
At the start: 1 part, among them J1 DA15_Plug

Commit message: Remove dsub
Parts:
- removed J1: DA15_Plug, Janelia:DSUB-15_Male_Vertical_SMD_09552296812741, symbol Janelia:DA15_Plug_Vertical_SMD_09552296812741
Changed lines of the file:
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@@
   (title_block
     (title "stepper_driver")
-    (date "2023-04-04")
+    (date "2023-04-06")
     (rev "2.0")
     (company "Howard Hughes Medical Institute")
   )
-  (symbol (lib_id "Janelia:DA15_Plug_Vertical_SMD_09552296812741") (at 129.54 90.17 0) (unit 1)
-    (in_bom yes) (on_board yes) (dnp no) (fields_autoplaced)
-    (property "Reference" "J1" (at 134.62 89.535 0)
-      (effects (font (size 1.27 1.27)) (justify left))
-    )
-    (property "Value" "DA15_Plug" (at 134.62 92.075 0)
-      (effects (font (size 1.27 1.27)) (justify left))
-    )
-    (property "Footprint" "Janelia:DSUB-15_Male_Vertical_SMD_09552296812741" (at 129.54 45.72 0)
-      (effects (font (size 1.27 1.27)) hide)
-    )
-    (property "Datasheet" " ~" (at 129.54 90.17 0)
-      (effects (font (size 1.27 1.27)) hide)
-    )
-    (property "Manufacturer" "HARTING" (at 129.54 53.34 0)
-      (effects (font (size 1.27 1.27)) hide)
-    )
-    (property "Manufacturer Part Number" "09552296812741" (at 129.54 48.26 0)
-      (effects (font (size 1.27 1.27)) hide)
-    )
-    (property "Description" "CONN D-SUB PLUG 15POS SMD SLDR" (at 129.54 50.8 0)
-      (effects (font (size 1.27 1.27)) hide)
-    )
-    (property "Vendor" "Digi-Key" (at 129.54 58.42 0)
-      (effects (font (size 1.27 1.27)) hide)
-    )
-    (property "Vendor Part Number" "1195-4008-1-ND" (at 129.54 55.88 0)
-      (effects (font (size 1.27 1.27)) hide)
-    )
-    (pin "1")
-    (pin "10")
-    (pin "11")
-    (pin "12")
-    (pin "13")
-    (pin "14")
-    (pin "15")
-    (pin "2")
-    (pin "3")
-    (pin "4")
-    (pin "5")
-    (pin "6")
-    (pin "7")
-    (pin "8")
-    (pin "9")
-    (instances
-      (project "stepper_driver"
-        (path "/cc457ebc-4af6-4663-b19f-8cb38f061cb4/f010267d-1aa0-4017-93cd-24b39ac4df1f"
-          (reference "J1") (unit 1)
-        )
-      )
-    )
-  )
 )
