File: stepper_driver/interface.kicad_sch (KiCad schematic)
At the start: 16 parts, among them J1 Conn_FFC_20_Pin_1mm_bottom-ZF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, J2 Conn_TERM_HDR_01x08_Pin_2.5MM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, U1 LVDS_4-4_HALF_DS91M040TSQE, U2 LVDS_4-4_HALF_DS91M040TSQE, U2 MAX6817

Commit message: Change 8 pin connector from surface mount to through hole
Parts:
- removed J2: Conn_TERM_HDR_01x08_Pin_2.5MM_Horizontal_SMD, Janelia:TERM_HDR_01x08_Pin_Horizontal_2.5MM_1778829, symbol Janelia:Conn_TERM_HDR_01x08_Pin_2.5MM_Horizontal_SMD
- added J2: Conn_TERM_HDR_01x08_Pin_2.5MM_Horizontal, Janelia:TERM_HDR_01x08_Pin_Horizontal_2.5MM_1778683, symbol Janelia:Conn_TERM_HDR_01x08_Pin_2.5MM_Horizontal
Connections:
- net A1: now also J2.3 (Pin_3)
- net A2: now also J2.4 (Pin_4)
- net B1: now also J2.5 (Pin_5)
- net B2: now also J2.6 (Pin_6)
- net GND: now also J2.1 (Pin_1), J2.8 (Pin_8)
- net REF: now also J2.7 (Pin_7)
- net REFR: now also J2.2 (Pin_2)
Changed lines of the file:
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@@
   (title_block
     (title "stepper_driver")
-    (date "2023-07-12")
+    (date "2023-07-13")
     (rev "2.0")
     (company "Howard Hughes Medical Institute")
@@
         (path "/cc457ebc-4af6-4663-b19f-8cb38f061cb4/25e66ddf-c258-4744-8ed9-64f4b44995b0"
           (reference "R2") (unit 1)
+        )
+      )
+    )
+  )
+  (symbol (lib_id "Janelia:Conn_TERM_HDR_01x08_Pin_2.5MM_Horizontal") (at 242.57 86.36 180) (unit 1)
+    (in_bom yes) (on_board yes) (dnp no) (fields_autoplaced)
+    (property "Reference" "J2" (at 243.84 85.09 0)
+      (effects (font (size 1.27 1.27)) (justify right))
+    )
+    (property "Value" "Conn_TERM_HDR_01x08_Pin_2.5MM_Horizontal" (at 242.57 73.66 0)
+      (effects (font (size 1.27 1.27)) hide)
+    )
+    (property "Footprint" "Janelia:TERM_HDR_01x08_Pin_Horizontal_2.5MM_1778683" (at 242.57 121.92 0)
+      (effects (font (size 1.27 1.27)) hide)
+    )
+    (property "Datasheet" "" (at 242.57 106.68 0)
+      (effects (font (size 1.27 1.27)) hide)
+    )
+    (property "Manufacturer" "Phoenix Contact" (at 242.57 119.38 0)
+      (effects (font (size 1.27 1.27)) hide)
+    )
+    (property "Manufacturer Part Number" "1778683" (at 242.57 114.3 0)
+      (effects (font (size 1.27 1.27)) hide)
+    )
+    (property "Description" "TERM BLOCK HDR 8POS 90DEG 2.5MM" (at 242.57 111.76 0)
+      (effects (font (size 1.27 1.27)) hide)
+    )
+    (property "Vendor" "Digi-Key" (at 242.57 116.84 0)
+      (effects (font (size 1.27 1.27)) hide)
+    )
+    (property "Vendor Part Number" "277-2314-1-ND" (at 242.57 109.22 0)
+      (effects (font (size 1.27 1.27)) hide)
+    )
+    (property "Sim.Enable" "0" (at 242.57 86.36 0)
+      (effects (font (size 1.27 1.27)) hide)
+    )
+    (pin "1")
+    (pin "2")
+    (pin "3")
+    (pin "4")
+    (pin "5")
+    (pin "6")
+    (pin "7")
+    (pin "8")
+    (instances
+      (project "stepper_driver"
+        (path "/cc457ebc-4af6-4663-b19f-8cb38f061cb4/25e66ddf-c258-4744-8ed9-64f4b44995b0"
+          (reference "J2") (unit 1)
         )
       )
@@
         )
       )
-    )
-  )
-  (symbol (lib_id "Janelia:Conn_TERM_HDR_01x08_Pin_2.5MM_Horizontal_SMD") (at 242.57 86.36 180) (unit 1)
-    (in_bom yes) (on_board yes) (dnp no) (fields_autoplaced)
-    (property "Reference" "J2" (at 243.84 85.09 0)
-      (effects (font (size 1.27 1.27)) (justify right))
-    )
-    (property "Value" "Conn_TERM_HDR_01x08_Pin_2.5MM_Horizontal_SMD" (at 242.57 73.66 0)
-      (effects (font (size 1.27 1.27)) hide)
-    )
-    (property "Footprint" "Janelia:TERM_HDR_01x08_Pin_Horizontal_2.5MM_1778829" (at 242.57 121.92 0)
-      (effects (font (size 1.27 1.27)) hide)
-    )
-    (property "Datasheet" "" (at 242.57 106.68 0)
-      (effects (font (size 1.27 1.27)) hide)
-    )
-    (property "Manufacturer" "Phoenix Contact" (at 242.57 119.38 0)
-      (effects (font (size 1.27 1.27)) hide)
-    )
-    (property "Manufacturer Part Number" "1778829" (at 242.57 114.3 0)
-      (effects (font (size 1.27 1.27)) hide)
-    )
-    (property "Description" "TERM BLOCK HDR 8POS 90DEG 2.5MM" (at 242.57 111.76 0)
-      (effects (font (size 1.27 1.27)) hide)
-    )
-    (property "Vendor" "Digi-Key" (at 242.57 116.84 0)
-      (effects (font (size 1.27 1.27)) hide)
-    )
-    (property "Vendor Part Number" "277-2321-1-ND" (at 242.57 109.22 0)
-      (effects (font (size 1.27 1.27)) hide)
-    )
-    (property "Sim.Enable" "0" (at 242.57 86.36 0)
-      (effects (font (size 1.27 1.27)) hide)
-    )
-    (pin "1")
-    (pin "2")
-    (pin "3")
-    (pin "4")
-    (pin "5")
-    (pin "6")
-    (pin "7")
-    (pin "8")
-    (instances
-      (project "stepper_driver"
-        (path "/cc457ebc-4af6-4663-b19f-8cb38f061cb4/25e66ddf-c258-4744-8ed9-64f4b44995b0"
-          (reference "J2") (unit 1)
-        )
-      )

Commit message: Route more tracks
Connections:
- net A1: now also J2.6 (Pin_6); no longer J2.3 (Pin_3)
- net A2: now also J2.5 (Pin_5); no longer J2.4 (Pin_4)
- net B1: now also J2.4 (Pin_4); no longer J2.5 (Pin_5)
- net B2: now also J2.3 (Pin_3); no longer J2.6 (Pin_6)
Changed lines of the file:
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@@
   (title_block
     (title "stepper_driver")
-    (date "2023-07-14")
+    (date "2023-07-18")
     (rev "2.0")
     (company "Howard Hughes Medical Institute")
@@
     (effects (font (size 1.27 1.27)) (justify right bottom))
   )
-  (label "A2" (at 234.95 86.36 180) (fields_autoplaced)
+  (label "A2" (at 234.95 83.82 180) (fields_autoplaced)
     (effects (font (size 1.27 1.27)) (justify right bottom))
   )
@@
     (effects (font (size 1.27 1.27)) (justify left bottom))
   )
-  (label "B1" (at 234.95 83.82 180) (fields_autoplaced)
+  (label "B1" (at 234.95 86.36 180) (fields_autoplaced)
     (effects (font (size 1.27 1.27)) (justify right bottom))
   )
@@
     (effects (font (size 1.27 1.27)) (justify left bottom))
   )
-  (label "A1" (at 234.95 88.9 180) (fields_autoplaced)
+  (label "A1" (at 234.95 81.28 180) (fields_autoplaced)
     (effects (font (size 1.27 1.27)) (justify right bottom))
   )
@@
     (effects (font (size 1.27 1.27)) (justify left bottom))
   )
-  (label "B2" (at 234.95 81.28 180) (fields_autoplaced)
-    (effects (font (size 1.27 1.27)) (justify right bottom))
-  )
+  (label "B2" (at 234.95 88.9 180) (fields_autoplaced)
+    (effects (font (size 1.27 1.27)) (justify right bottom))
+  )
